File: Hardware/Power Board/LS_PWR_STAGE.kicad_sch (KiCad schematic)
At the start: 62 parts, among them IC1 SN6507DGQR, IC2 UCC21737-Q1, Q10 AO3400A, Q11 G3R40MT12J, Q12 AO3400A, Q13 G3R40MT12J, Q4 AO3400A, Q9 G3R40MT12J, T1 782100_35JVC, U1 L78M15, U5 LM7905S

Commit message: Finished intial LV board connector routing, going to tear up current sense and redo
Parts:
- Q11, Q13, Q9: footprint SamacSys_Parts:G3R40MT12J -> G3R40MT12J
- T1: footprint SamacSys_Parts:78210035JVC -> 78210035JVC
- U3: renamed from U5; value LM7905S -> LM7905_TO220
Connections:
- net COM is gone; now on net FET_SOURCE: C10.2, C114.2, C33.2, C34.1, C35.2, C36.1, C40.1, C49.1, C50.1, C58.1, C59.1, C61.1, C64.1, C69.1, C93.1, D14.2 (A), D15.1 (K), IC2.1 (ASC), IC2.2 (OC), IC2.3 (COM), Q11.2 (KS), Q13.2 (KS), Q9.2 (KS), T1.5 (SEC_2), U1.2 (GND), U3.1 (GND)
Changed lines of the file:
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@@
   (junction (at 190.5 88.265) (diameter 0) (color 0 0 0 0)
   )
+  (junction (at 353.06 194.945) (diameter 0) (color 0 0 0 0)
+  )
   (junction (at 171.45 159.385) (diameter 0) (color 0 0 0 0)
   )
@@
   (junction (at 172.085 74.295) (diameter 0) (color 0 0 0 0)
   )
+  (junction (at 345.44 194.945) (diameter 0) (color 0 0 0 0)
+  )
+  (junction (at 204.47 194.945) (diameter 0) (color 0 0 0 0)
+  )
   (junction (at 190.5 57.785) (diameter 0) (color 0 0 0 0)
   )
@@
   (junction (at 303.53 149.225) (diameter 0) (color 0 0 0 0)
   )
+  (junction (at 273.05 194.945) (diameter 0) (color 0 0 0 0)
+  )
   (junction (at 283.21 213.995) (diameter 0) (color 0 0 0 0)
   )
@@
   (junction (at 176.53 151.765) (diameter 0) (color 0 0 0 0)
   )
+  (junction (at 280.67 194.945) (diameter 0) (color 0 0 0 0)
+  )
   (junction (at 345.44 191.135) (diameter 0) (color 0 0 0 0)
   )
@@
   (junction (at 273.05 191.135) (diameter 0) (color 0 0 0 0)
   )
+  (junction (at 196.85 194.945) (diameter 0) (color 0 0 0 0)
+  )
   (junction (at 159.385 57.785) (diameter 0) (color 0 0 0 0)
   )
@@
     (stroke (width 0) (type default))
   )
-  (wire (pts (xy 280.67 191.135) (xy 280.67 224.79))
+  (wire (pts (xy 280.67 191.135) (xy 280.67 194.945))
     (stroke (width 0) (type default))
   )
@@
     (stroke (width 0) (type default))
   )
+  (wire (pts (xy 273.05 194.945) (xy 280.67 194.945))
+    (stroke (width 0) (type default))
+  )
   (wire (pts (xy 353.06 74.295) (xy 354.965 74.295))
     (stroke (width 0) (type default))
   )
+  (wire (pts (xy 353.06 194.945) (xy 353.06 224.79))
+    (stroke (width 0) (type default))
+  )
   (wire (pts (xy 335.28 88.265) (xy 353.06 88.265))
     (stroke (width 0) (type default))
@@
     (stroke (width 0) (type default))
   )
-  (wire (pts (xy 204.47 191.135) (xy 204.47 224.79))
+  (wire (pts (xy 204.47 191.135) (xy 204.47 194.945))
     (stroke (width 0) (type default))
   )
@@
     (stroke (width 0) (type default))
   )
-  (wire (pts (xy 353.06 191.135) (xy 353.06 224.79))
+  (wire (pts (xy 353.06 191.135) (xy 353.06 194.945))
     (stroke (width 0) (type default))
   )
@@
     (stroke (width 0) (type default))
   )
+  (wire (pts (xy 345.44 194.945) (xy 353.06 194.945))
+    (stroke (width 0) (type default))
+  )
   (wire (pts (xy 194.945 194.945) (xy 196.85 194.945))
     (stroke (width 0) (type default))
@@
     (stroke (width 0) (type default))
   )
+  (wire (pts (xy 280.67 194.945) (xy 280.67 224.79))
+    (stroke (width 0) (type default))
+  )
   (wire (pts (xy 204.47 224.79) (xy 176.53 224.79))
     (stroke (width 0) (type default))
@@
     (stroke (width 0) (type default))
   )
+  (wire (pts (xy 196.85 194.945) (xy 204.47 194.945))
+    (stroke (width 0) (type default))
+  )
   (wire (pts (xy 350.52 191.135) (xy 347.98 191.135))
     (stroke (width 0) (type default))
@@
     (stroke (width 0) (type default))
   )
+  (wire (pts (xy 204.47 194.945) (xy 204.47 224.79))
+    (stroke (width 0) (type default))
+  )
   (wire (pts (xy 106.045 86.995) (xy 106.045 88.265))
     (stroke (width 0) (type default))
@@
       (effects (font (size 0.75 0.75)) (justify right))
     )
-    (property "Footprint" "SamacSys_Parts:G3R40MT12J" (at 209.55 172.085 0)
+    (property "Footprint" "G3R40MT12J" (at 209.55 172.085 0)
       (effects (font (size 1.27 1.27)) (justify left) hide)
     )
@@
       (effects (font (size 0.75 0.75)))
     )
-    (property "Footprint" "SamacSys_Parts:78210035JVC" (at 132.715 69.215 0)
+    (property "Footprint" "78210035JVC" (at 132.715 69.215 0)
       (effects (font (size 1.27 1.27)) (justify left) hide)
     )
@@
       (effects (font (size 0.75 0.75)) (justify right))
     )
-    (property "Footprint" "SamacSys_Parts:G3R40MT12J" (at 358.14 172.085 0)
+    (property "Footprint" "G3R40MT12J" (at 358.14 172.085 0)
       (effects (font (size 1.27 1.27)) (justify left) hide)
     )
@@
       (effects (font (size 0.75 0.75)) (justify right))
     )
-    (property "Footprint" "SamacSys_Parts:G3R40MT12J" (at 285.75 172.085 0)
+    (property "Footprint" "G3R40MT12J" (at 285.75 172.085 0)
       (effects (font (size 1.27 1.27)) (justify left) hide)
     )
@@
   (symbol (lib_id "Regulator_Linear:LM7905_TO220") (at 254 88.265 0) (unit 1)
     (in_bom yes) (on_board yes) (dnp no) (fields_autoplaced)
-    (property "Reference" "U5" (at 254 92.71 0)
-      (effects (font (size 0.75 0.75)))
+    (property "Reference" "U3" (at 250.19 91.44 0)
+      (effects (font (size 1.27 1.27)))
     )
-    (property "Value" "LM7905S" (at 254 95.25 0)
-      (effects (font (size 0.75 0.75)))
+    (property "Value" "LM7905_TO220" (at 254 91.44 0)
+      (effects (font (size 1.27 1.27)) (justify left))
     )
     (property "Footprint" "Package_TO_SOT_SMD:TO-263-3_TabPin2" (at 254 93.345 0)
@@
       (project "Power Board"
         (path "/6be5afcf-5319-4edd-874e-36cb4fffe262/6614681d-fa8a-47d6-92cc-5feb6bb30852"
-          (reference "U5") (unit 1)
+          (reference "U3") (unit 1)
         )
         (path "/6be5afcf-5319-4edd-874e-36cb4fffe262/1499af7b-9903-43ec-b2cd-1e9dc72da420"
-          (reference "U3") (unit 1)
+          (reference "U5") (unit 1)
         )
         (path "/6be5afcf-5319-4edd-874e-36cb4fffe262/92924a04-f6bb-42dd-aa65-b0f7ec7a97f7"
